File: Hardware/Beecounter.kicad_sch (KiCad schematic)
At the start: 141 parts, among them J1 Conn_01x03, J10 Conn_01x03, J11 Conn_01x03, J12 Conn_01x03, J13 Conn_01x03, J14 Conn_01x03, J15 Conn_02x20_Odd_Even, J2 Conn_01x03, J3 Conn_01x03, J4 Conn_01x03, J5 Conn_01x03, J6 Conn_01x03, J7 Conn_01x03, J8 Conn_01x03, J9 Conn_01x03, U1 LM393, U10 LM393, U11 H2010, U12 LM393, U13 H2010, U14 LM393, U15 H2010, U16 LM393, U17 H2010, U18 LM393, U19 H2010, U2 H2010, U20 LM393, U21 H2010, U22 LM393, U23 H2010, U24 LM393, U25 H2010, U26 LM393, U27 H2010, U28 LM393, U3 H2010, U4 LM393, U5 H2010, U6 LM393, U7 H2010, U8 LM393, U9 H2010

Commit message: Exchanged pin 13 with 32 and 11 with 36
Connections:
- net at D1.1 (K), J1.2 (Pin_2), U1.1: now also J15.36 (Pin_36); no longer J15.11 (Pin_11)
- net at D10.1 (K), J10.2 (Pin_2), J15.16 (Pin_16)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: no longer D3.1 (K), J15.18 (Pin_18), J3.2 (Pin_2), U6.1
- net at D2.1 (K), J2.2 (Pin_2), U4.1: now also J15.32 (Pin_32); no longer J15.13 (Pin_13)
- new net: D3.1 (K), J15.18 (Pin_18), J3.2 (Pin_2), U6.1
Changed lines of the file:
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@@
 	)
 	(junction
-		(at 176.53 676.91)
-		(diameter 0)
-		(color 0 0 0 0)
-	)
-	(junction
 		(at 118.11 554.99)
 		(diameter 0)
@@
 	)
 	(junction
-		(at 179.07 638.81)
-		(diameter 0)
-		(color 0 0 0 0)
-	)
-	(junction
 		(at 382.27 300.99)
 		(diameter 0)
@@
 	)
 	(junction
-		(at 173.99 676.91)
-		(diameter 0)
-		(color 0 0 0 0)
-	)
-	(junction
 		(at 118.11 59.69)
 		(diameter 0)
@@
 	(wire
 		(pts
-			(xy 54.61 140.97) (xy 54.61 702.31)
+			(xy 54.61 140.97) (xy 54.61 656.59)
 		)
 		(stroke
@@
 	(wire
 		(pts
-			(xy 168.91 632.46) (xy 168.91 664.21)
+			(xy 168.91 633.73) (xy 168.91 664.21)
 		)
 		(stroke
@@
 	(wire
 		(pts
-			(xy 313.69 656.59) (xy 171.45 656.59)
+			(xy 313.69 654.05) (xy 171.45 654.05)
 		)
 		(stroke
@@
 	(wire
 		(pts
-			(xy 63.5 223.52) (xy 63.5 638.81)
+			(xy 63.5 223.52) (xy 63.5 643.89)
 		)
 		(stroke
@@
 	(wire
 		(pts
-			(xy 73.66 388.62) (xy 73.66 632.46)
+			(xy 73.66 388.62) (xy 73.66 633.73)
 		)
 		(stroke
@@
 	(wire
 		(pts
-			(xy 80.01 621.03) (xy 189.23 621.03)
+			(xy 80.01 628.65) (xy 189.23 628.65)
 		)
 		(stroke
@@
 	(wire
 		(pts
-			(xy 189.23 621.03) (xy 189.23 664.21)
+			(xy 189.23 628.65) (xy 189.23 664.21)
 		)
 		(stroke
@@
 	(wire
 		(pts
-			(xy 173.99 624.84) (xy 173.99 664.21)
-		)
-		(stroke
-			(width 0)
-			(type default)
-		)
-	)
-	(wire
-		(pts
-			(xy 179.07 638.81) (xy 179.07 631.19)
+			(xy 173.99 622.3) (xy 173.99 664.21)
 		)
 		(stroke
@@
 	(wire
 		(pts
-			(xy 288.29 624.84) (xy 173.99 624.84)
+			(xy 288.29 622.3) (xy 173.99 622.3)
 		)
 		(stroke
@@
 	(wire
 		(pts
+			(xy 54.61 656.59) (xy 199.39 656.59)
+		)
+		(stroke
+			(width 0)
+			(type default)
+		)
+	)
+	(wire
+		(pts
 			(xy 426.72 476.25) (xy 426.72 466.09)
 		)
@@
 	(wire
 		(pts
-			(xy 67.31 643.89) (xy 186.69 643.89)
+			(xy 67.31 636.27) (xy 186.69 636.27)
 		)
 		(stroke
@@
 	(wire
 		(pts
+			(xy 204.47 664.21) (xy 204.47 650.24)
+		)
+		(stroke
+			(width 0)
+			(type default)
+		)
+	)
+	(wire
+		(pts
 			(xy 184.15 694.69) (xy 184.15 676.91)
 		)
@@
 	(wire
 		(pts
-			(xy 186.69 683.26) (xy 186.69 676.91)
+			(xy 186.69 684.53) (xy 186.69 676.91)
 		)
 		(stroke
@@
 	(wire
 		(pts
-			(xy 326.39 554.99) (xy 326.39 683.26)
+			(xy 326.39 554.99) (xy 326.39 684.53)
 		)
 		(stroke
@@
 	(wire
 		(pts
-			(xy 179.07 676.91) (xy 179.07 697.23)
+			(xy 179.07 676.91) (xy 179.07 689.61)
 		)
 		(stroke
@@
 	(wire
 		(pts
-			(xy 67.31 306.07) (xy 67.31 643.89)
+			(xy 67.31 306.07) (xy 67.31 636.27)
 		)
 		(stroke
@@
 	(wire
 		(pts
-			(xy 48.26 62.23) (xy 48.26 698.5)
+			(xy 57.15 62.23) (xy 57.15 650.24)
 		)
 		(stroke
@@
 	(wire
 		(pts
-			(xy 179.07 638.81) (xy 181.61 638.81)
+			(xy 63.5 643.89) (xy 181.61 643.89)
 		)
 		(stroke
@@
 	(wire
 		(pts
-			(xy 294.64 138.43) (xy 294.64 697.23)
+			(xy 294.64 138.43) (xy 294.64 689.61)
 		)
 		(stroke
@@
 	(wire
 		(pts
-			(xy 166.37 651.51) (xy 166.37 660.4)
-		)
-		(stroke
-			(width 0)
-			(type default)
-		)
-	)
-	(wire
-		(pts
 			(xy 367.03 383.54) (xy 381 383.54)
 		)
@@
 	(wire
 		(pts
-			(xy 104.14 651.51) (xy 166.37 651.51)
+			(xy 102.87 660.4) (xy 166.37 660.4)
 		)
 		(stroke
@@
 	(wire
 		(pts
-			(xy 173.99 676.91) (xy 173.99 698.5)
-		)
-		(stroke
-			(width 0)
-			(type default)
-		)
-	)
-	(wire
-		(pts
 			(xy 419.1 388.62) (xy 426.72 388.62)
 		)
@@
 	(wire
 		(pts
-			(xy 73.66 632.46) (xy 168.91 632.46)
+			(xy 73.66 633.73) (xy 168.91 633.73)
 		)
 		(stroke
@@
 	(wire
 		(pts
-			(xy 300.99 220.98) (xy 300.99 631.19)
+			(xy 300.99 220.98) (xy 300.99 638.81)
 		)
 		(stroke
@@
 	(wire
 		(pts
-			(xy 176.53 676.91) (xy 176.53 702.31)
-		)
-		(stroke
-			(width 0)
-			(type default)
-		)
-	)
-	(wire
-		(pts
 			(xy 499.11 113.03) (xy 499.11 115.57)
 		)
@@
 	(wire
 		(pts
-			(xy 313.69 386.08) (xy 313.69 656.59)
+			(xy 313.69 386.08) (xy 313.69 654.05)
 		)
 		(stroke
@@
 	(wire
 		(pts
-			(xy 294.64 697.23) (xy 179.07 697.23)
+			(xy 294.64 689.61) (xy 179.07 689.61)
 		)
 		(stroke
@@
 	(wire
 		(pts
-			(xy 171.45 656.59) (xy 171.45 664.21)
+			(xy 171.45 654.05) (xy 171.45 664.21)
+		)
+		(stroke
+			(width 0)
+			(type default)
+		)
+	)
+	(wire
+		(pts
+			(xy 199.39 664.21) (xy 199.39 656.59)
 		)
 		(stroke
@@
 	(wire
 		(pts
-			(xy 179.07 664.21) (xy 179.07 638.81)
+			(xy 179.07 638.81) (xy 179.07 664.21)
 		)
 		(stroke
@@
 	(wire
 		(pts
-			(xy 63.5 638.81) (xy 179.07 638.81)
-		)
-		(stroke
-			(width 0)
-			(type default)
-		)
-	)
-	(wire
-		(pts
 			(xy 439.42 91.44) (xy 459.74 91.44)
 		)
@@
 	(wire
 		(pts
-			(xy 326.39 683.26) (xy 186.69 683.26)
+			(xy 326.39 684.53) (xy 186.69 684.53)
 		)
 		(stroke
@@
 	(wire
 		(pts
-			(xy 186.69 643.89) (xy 186.69 664.21)
+			(xy 186.69 636.27) (xy 186.69 664.21)
 		)
 		(stroke
@@
 	(wire
 		(pts
+			(xy 102.87 560.07) (xy 104.14 560.07)
+		)
+		(stroke
+			(width 0)
+			(type default)
+		)
+	)
+	(wire
+		(pts
 			(xy 173.99 91.44) (xy 186.69 91.44)
 		)
@@
 	(wire
 		(pts
-			(xy 288.29 62.23) (xy 288.29 624.84)
+			(xy 288.29 62.23) (xy 288.29 622.3)
 		)
 		(stroke
@@
 	(wire
 		(pts
-			(xy 179.07 631.19) (xy 300.99 631.19)
+			(xy 179.07 638.81) (xy 300.99 638.81)
 		)
 		(stroke
@@
 	(wire
 		(pts
-			(xy 80.01 474.98) (xy 80.01 621.03)
+			(xy 80.01 474.98) (xy 80.01 628.65)
 		)
 		(stroke
@@
 	(wire
 		(pts
-			(xy 181.61 664.21) (xy 181.61 638.81)
+			(xy 181.61 664.21) (xy 181.61 643.89)
 		)
 		(stroke
@@
 	(wire
 		(pts
-			(xy 173.99 698.5) (xy 48.26 698.5)
+			(xy 57.15 650.24) (xy 204.47 650.24)
 		)
 		(stroke
@@
 	(wire
 		(pts
-			(xy 104.14 560.07) (xy 104.14 651.51)
+			(xy 102.87 560.07) (xy 102.87 660.4)
 		)
 		(stroke
@@
 	(wire
 		(pts
-			(xy 176.53 702.31) (xy 54.61 702.31)
-		)
-		(stroke
-			(width 0)
-			(type default)
-		)
-	)
-	(wire
-		(pts
 			(xy 433.07 547.37) (xy 458.47 547.37)
 		)
@@
 	(wire
 		(pts
-			(xy 48.26 62.23) (xy 133.35 62.23)
+			(xy 57.15 62.23) (xy 133.35 62.23)
 		)
 		(stroke

Commit message: Added connector for HX711 (H-bridge) and ADC ADS1115
Parts:
- added J16: Conn_01x04, Connector_PinSocket_2.54mm:PinSocket_1x04_P2.54mm_Vertical, symbol Connector_Generic:Conn_01x04
- added J17: Conn_01x10, Connector_PinHeader_2.54mm:PinHeader_1x10_P2.54mm_Vertical, symbol Connector_Generic:Conn_01x10
- added J18: Conn_02x04_Odd_Even, symbol Connector_Generic:Conn_02x04_Odd_Even
Connections:
- net GND: now also J16.4 (Pin_4), J17.2 (Pin_2), J18.1 (Pin_1), J18.3 (Pin_3), J18.5 (Pin_5), J18.7 (Pin_7)
- net at J15.2 (Pin_2): now also J16.1 (Pin_1), J17.1 (Pin_1)
- net at J15.29 (Pin_29): now also J16.3 (Pin_3)
- net at J15.3 (Pin_3): now also J17.4 (Pin_4)
- net at J15.31 (Pin_31): now also J16.2 (Pin_2)
- net at J15.5 (Pin_5): now also J17.3 (Pin_3), J17.5 (Pin_5)
- new net: J17.10 (Pin_10), J18.8 (Pin_8)
- new net: J17.7 (Pin_7), J18.2 (Pin_2)
- new net: J17.8 (Pin_8), J18.4 (Pin_4)
- new net: J17.9 (Pin_9), J18.6 (Pin_6)
